File: prototyping/PCB_prototype/Masimo_cable_tester_1.kicad_sch (KiCad schematic)
At the start: 28 parts, among them J1 Touchscreen HMI, J10 MCU Board Power, J16 Debug Connections, J17 Banana Jack, J2 Curiosity Nano AVR128DB48, J3 Conn_01x28_Socket, J4 Barrel Jack 9V, J5 MicroSD PinHeader, J6 SFML-110-02-L-D-A, J7 HMI Power Toggle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

Commit message: Updated Prototype Schematic and PCB
Parts:
- added Q1: 2N3904, Package_TO_SOT_THT:TO-92_Inline, symbol Transistor_BJT:2N3904
- added R2: 1.5kΩ 1/4W, KiCad Symbols and Footprints:RES_ERA8AEB152V, symbol Device:R
Connections:
- net 5V: now also D2.K, U1.1
- net GND: now also Q1.1 (E); no longer D2.A, U1.8
- net BJ1: no longer names the net of J17.1 (Pin_1), U1.2
- net BJ2: no longer names the net of J17.2 (Pin_2), U1.3
- net CD: no longer names the net of J2.9 (Pin_9), J5.8 (Pin_8), R1.2
- net CLK: no longer names the net of J2.13 (Pin_13), J5.4 (Pin_4)
- net CS: no longer names the net of J2.10 (Pin_10), J5.7 (Pin_7)
- net DI: no longer names the net of J2.11 (Pin_11), J5.6 (Pin_6)
- net DO: no longer names the net of J2.12 (Pin_12), J5.5 (Pin_5)
- removed net RSig: D2.K, J2.23 (Pin_23), U1.1
- net Rx1: no longer names the net of J1.3 (Pin_3), J2.7 (Pin_7)
- net Rx2: no longer names the net of J16.3 (Pin_3), J2.3 (Pin_3)
- net Tx1: no longer names the net of J1.2 (Pin_2), J2.8 (Pin_8)
- net Tx2: no longer names the net of J16.2 (Pin_2), J2.4 (Pin_4)
- new net: Q1.2 (B), R2.2
- new net: D2.A, Q1.3 (C), U1.8
- new net: J2.23 (Pin_23), R2.1
Other:
- note added: "20 Pin Connector"
- note added: "Cable tester - Prototype PCB"
- note removed: "20-Pin Connector"
- moved on the sheet: C1, C2, D2, J1, J10, J16, J17, J2, J3, J4, J5, J6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
