File: prototyping/PCB_prototype/Masimo_cable_tester_1.kicad_pcb (KiCad board)
At the start: 2 copper layers, 80 x 90 mm, 30 parts, among them J1 Touchscreen HMI, J10 MCU Board Power, J16 Debug Connections, J17 Banana Jack, J2 Curiosity Nano AVR128DB48, J3 Conn_01x28_Socket, J4 Barrel Jack 9V, J5 MicroSD PinHeader, J6 SFML-110-02-L-D-A, J7 HMI Power Toggle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

Commit message: Changed spacing to account for overhang.
Parts:
- moved J7 6.50 mm to (83.5, 58.0)
- moved J1 6.50 mm to (83.5, 78.3)
- moved J16 6.50 mm to (83.5, 126.5)
- moved J5 6.50 mm to (83.5, 108.8)
Routing:
- net 5V: track 153.3 -> 196.9 mm
- net VBUS 5V: track 24.2 -> 31.6 mm
- net Net-(J2-Pin_10): track 15.9 -> 22.4 mm
- net UPDI: track 71.1 -> 77.6 mm
- net Net-(J2-Pin_9): track 16.0 -> 22.5 mm
- net Net-(J2-Pin_13): track 15.9 -> 22.4 mm
- net Net-(J2-Pin_12): track 15.9 -> 22.4 mm
- net Net-(J2-Pin_11): track 15.9 -> 22.4 mm
- net Net-(J16-Pin_3): track 64.3 -> 70.8 mm
- net Net-(J1-Pin_3): track 7.78 -> 14.3 mm
- net Net-(J1-Pin_2): track 7.78 -> 14.3 mm
- net Net-(J16-Pin_2): track 64.8 -> 71.2 mm
- net GND: track 200.2 -> 206.1 mm
- net Net-(J1-Pin_1): track 18.7 -> 19.4 mm
