File: prototyping/PCB_prototype_THT/Masimo THT Prototype design/Masimo TH Design.kicad_pcb (KiCad board)
At the start: 2 copper layers, 100 x 66 mm, 30 parts, among them J1 Touchscreen HMI, J10 MCU Board Power, J11 SFML-110-T1-S-D, J16 Debug Connections, J17 Banana Jack, J2 Curiosity Nano AVR128DB48, J3 Conn_01x28_Socket, J4 Barrel Jack 9V, J5 MicroSD PinHeader, J7 HMI Power Toggle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

Commit message: Updated THT Prototype PCB
Updates to the through hole prototype PCB design
Connections:
- J4 pad B: unconnected-(J4-PadB) -> GND
Other:
- outline, holes or cut-outs redrawn
