File: prototyping/PCB_prototype_THT/Masimo THT Prototype design/Masimo TH Design.kicad_sch (KiCad schematic)
At the start: 30 parts, among them J1 Touchscreen HMI, J10 MCU Board Power, J11 SFML-110-T1-S-D, J16 Debug Connections, J17 Banana Jack, J2 Curiosity Nano AVR128DB48, J3 Conn_01x28_Socket, J4 Barrel Jack 9V, J5 MicroSD PinHeader, J7 HMI Power Toggle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

Commit message: Updated THT Prototype PCB
Updates to the through hole prototype PCB design
Connections:
- net GND: now also J4.B
- no-connect marks 22 -> 31
Changed lines of the file:
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@@
 	)
 	(junction
+		(at 187.96 146.05)
+		(diameter 0)
+		(color 0 0 0 0)
+	)
+	(junction
 		(at 200.66 29.21)
 		(diameter 0)
@@
 	)
 	(no_connect
+		(at 257.81 86.36)
+	)
+	(no_connect
 		(at 101.6 102.87)
 	)
 	(no_connect
-		(at 186.69 148.59)
+		(at 267.97 86.36)
+	)
+	(no_connect
+		(at 265.43 60.96)
+	)
+	(no_connect
+		(at 267.97 60.96)
+	)
+	(no_connect
+		(at 260.35 86.36)
 	)
 	(no_connect
@@
 	)
 	(no_connect
+		(at 262.89 60.96)
+	)
+	(no_connect
 		(at 101.6 92.71)
 	)
@@
 	)
 	(no_connect
+		(at 260.35 60.96)
+	)
+	(no_connect
 		(at 101.6 128.27)
 	)
@@
 	)
 	(no_connect
+		(at 257.81 60.96)
+	)
+	(no_connect
 		(at 41.91 114.3)
 	)
 	(no_connect
+		(at 262.89 86.36)
+	)
+	(no_connect
 		(at 123.19 128.27)
 	)
 	(no_connect
+		(at 265.43 86.36)
+	)
+	(no_connect
 		(at 101.6 120.65)
 	)
@@
 	(wire
 		(pts
+			(xy 187.96 146.05) (xy 186.69 146.05)
+		)
+		(stroke
+			(width 0)
+			(type default)
+		)
+	)
+	(wire
+		(pts
 			(xy 199.39 77.47) (xy 200.66 77.47)
 		)
@@
 	(wire
 		(pts
-			(xy 191.77 146.05) (xy 186.69 146.05)
+			(xy 191.77 146.05) (xy 187.96 146.05)
 		)
 		(stroke
@@
 	(wire
 		(pts
+			(xy 187.96 148.59) (xy 187.96 146.05)
+		)
+		(stroke
+			(width 0)
+			(type default)
+		)
+	)
+	(wire
+		(pts
 			(xy 41.91 116.84) (xy 43.18 116.84)
 		)
@@
 	(wire
 		(pts
+			(xy 187.96 148.59) (xy 186.69 148.59)
+		)
+		(stroke
+			(width 0)
+			(type default)
+		)
+	)
+	(wire
+		(pts
 			(xy 158.75 62.23) (xy 152.4 62.23)
 		)
@@
 		(dnp no)
 		(property "Reference" "J11"
-			(at 271.78 74.9301 90)
+			(at 272.034 73.66 90)
 			(effects
 				(font
@@
 		)
 		(property "Value" "SFML-110-T1-S-D"
-			(at 271.78 72.3901 90)
+			(at 246.888 73.914 90)
 			(effects
 				(font
@@
 		(dnp no)
 		(property "Reference" "U1"
-			(at 94.742 153.67 0)
+			(at 74.93 158.75 0)
 			(effects
 				(font

Commit message: Changes to Final board design
Re-routed the DO from microSD to MCU (No more level shifter), added a 5V line to pin 20 so that port C will be powered. Fixed other minor issues after running DRC on layout design.
Parts:
- R1, R10, R11, R12, R2, R3, R4, R5, R6, R7, R8, R9: footprint Resistor_THT:R_Axial_DIN0207_L6.3mm_D2.5mm_P7.62mm_Horizontal -> Resistor_THT:R_Axial_DIN0207_L6.3mm_D2.5mm_P10.16mm_Horizontal
Changed lines of the file:
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@@
 			)
 		)
-		(property "Footprint" "Resistor_THT:R_Axial_DIN0207_L6.3mm_D2.5mm_P7.62mm_Horizontal"
+		(property "Footprint" "Resistor_THT:R_Axial_DIN0207_L6.3mm_D2.5mm_P10.16mm_Horizontal"
 			(at 195.58 39.878 90)
 			(effects
@@
 			)
 		)
-		(property "Footprint" "Resistor_THT:R_Axial_DIN0207_L6.3mm_D2.5mm_P7.62mm_Horizontal"
+		(property "Footprint" "Resistor_THT:R_Axial_DIN0207_L6.3mm_D2.5mm_P10.16mm_Horizontal"
 			(at 195.58 60.198 90)
 			(effects
@@
 			)
 		)
-		(property "Footprint" "Resistor_THT:R_Axial_DIN0207_L6.3mm_D2.5mm_P7.62mm_Horizontal"
+		(property "Footprint" "Resistor_THT:R_Axial_DIN0207_L6.3mm_D2.5mm_P10.16mm_Horizontal"
 			(at 195.58 99.568 90)
 			(effects
@@
 			)
 		)
-		(property "Footprint" "Resistor_THT:R_Axial_DIN0207_L6.3mm_D2.5mm_P7.62mm_Horizontal"
+		(property "Footprint" "Resistor_THT:R_Axial_DIN0207_L6.3mm_D2.5mm_P10.16mm_Horizontal"
 			(at 195.58 70.358 90)
 			(effects
@@
 			)
 		)
-		(property "Footprint" "Resistor_THT:R_Axial_DIN0207_L6.3mm_D2.5mm_P7.62mm_Horizontal"
+		(property "Footprint" "Resistor_THT:R_Axial_DIN0207_L6.3mm_D2.5mm_P10.16mm_Horizontal"
 			(at 195.58 109.728 90)
 			(effects
@@
 			)
 		)
-		(property "Footprint" "Resistor_THT:R_Axial_DIN0207_L6.3mm_D2.5mm_P7.62mm_Horizontal"
+		(property "Footprint" "Resistor_THT:R_Axial_DIN0207_L6.3mm_D2.5mm_P10.16mm_Horizontal"
 			(at 195.58 79.248 90)
 			(effects
@@
 			)
 		)
-		(property "Footprint" "Resistor_THT:R_Axial_DIN0207_L6.3mm_D2.5mm_P7.62mm_Horizontal"
+		(property "Footprint" "Resistor_THT:R_Axial_DIN0207_L6.3mm_D2.5mm_P10.16mm_Horizontal"
 			(at 50.292 93.98 90)
 			(effects
@@
 			)
 		)
-		(property "Footprint" "Resistor_THT:R_Axial_DIN0207_L6.3mm_D2.5mm_P7.62mm_Horizontal"
+		(property "Footprint" "Resistor_THT:R_Axial_DIN0207_L6.3mm_D2.5mm_P10.16mm_Horizontal"
 			(at 46.482 132.08 90)
 			(effects
@@
 			)
 		)
-		(property "Footprint" "Resistor_THT:R_Axial_DIN0207_L6.3mm_D2.5mm_P7.62mm_Horizontal"
+		(property "Footprint" "Resistor_THT:R_Axial_DIN0207_L6.3mm_D2.5mm_P10.16mm_Horizontal"
 			(at 195.58 30.988 90)
 			(effects
@@
 			)
 		)
-		(property "Footprint" "Resistor_THT:R_Axial_DIN0207_L6.3mm_D2.5mm_P7.62mm_Horizontal"
+		(property "Footprint" "Resistor_THT:R_Axial_DIN0207_L6.3mm_D2.5mm_P10.16mm_Horizontal"
 			(at 195.58 89.408 90)
 			(effects
@@
 			)
 		)
-		(property "Footprint" "Resistor_THT:R_Axial_DIN0207_L6.3mm_D2.5mm_P7.62mm_Horizontal"
+		(property "Footprint" "Resistor_THT:R_Axial_DIN0207_L6.3mm_D2.5mm_P10.16mm_Horizontal"
 			(at 195.58 119.888 90)
 			(effects
@@
 			)
 		)
-		(property "Footprint" "Resistor_THT:R_Axial_DIN0207_L6.3mm_D2.5mm_P7.62mm_Horizontal"
+		(property "Footprint" "Resistor_THT:R_Axial_DIN0207_L6.3mm_D2.5mm_P10.16mm_Horizontal"
 			(at 195.58 50.038 90)
 			(effects
